File: codec.kicad_sch (KiCad schematic)
At the start: 16 parts, among them J3 Conn_01x03_Pin, U8 CM108AH, U9 93C46

Commit message: Assign footprints to devices
Parts:
- C11, C12, C13, C14, C15, C18, C19: footprint (none) -> Capacitor_SMD:C_0201_0603Metric
- D3, D4: footprint (none) -> LED_SMD:LED_0201_0603Metric
- J3: footprint (none) -> Connector_PinHeader_1.00mm:PinHeader_1x03_P1.00mm_Vertical_SMD_Pin1Left
- R15, R16, R17, R18: footprint (none) -> Resistor_SMD:R_0201_0603Metric
- U8: footprint CM108AH:QFP50P900X900X160-48N -> Package_QFP:LQFP-48_7x7mm_P0.5mm
- U9: footprint (none) -> Package_SO:SOIC-8_3.9x4.9mm_P1.27mm
Changed lines of the file:
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@@
 			)
 		)
-		(property "Footprint" ""
+		(property "Footprint" "Capacitor_SMD:C_0201_0603Metric"
 			(at 230.8352 85.09 0)
 			(effects
@@
 			)
 		)
-		(property "Footprint" ""
+		(property "Footprint" "LED_SMD:LED_0201_0603Metric"
 			(at 213.36 130.81 0)
 			(effects
@@
 			)
 		)
-		(property "Footprint" ""
+		(property "Footprint" "Resistor_SMD:R_0201_0603Metric"
 			(at 73.914 162.814 90)
 			(effects
@@
 			)
 		)
-		(property "Footprint" ""
+		(property "Footprint" "Capacitor_SMD:C_0201_0603Metric"
 			(at 191.4652 68.58 0)
 			(effects
@@
 			)
 		)
-		(property "Footprint" ""
+		(property "Footprint" "Resistor_SMD:R_0201_0603Metric"
 			(at 205.994 143.764 90)
 			(effects
@@
 			)
 		)
-		(property "Footprint" "CM108AH:QFP50P900X900X160-48N"
+		(property "Footprint" "Package_QFP:LQFP-48_7x7mm_P0.5mm"
 			(at 127.762 33.274 0)
 			(effects
@@
 			)
 		)
-		(property "Footprint" ""
+		(property "Footprint" "Capacitor_SMD:C_0201_0603Metric"
 			(at 180.0352 68.58 0)
 			(effects
@@
 			)
 		)
-		(property "Footprint" ""
+		(property "Footprint" "Package_SO:SOIC-8_3.9x4.9mm_P1.27mm"
 			(at 173.99 106.68 0)
 			(effects
@@
 			)
 		)
-		(property "Footprint" ""
+		(property "Footprint" "Capacitor_SMD:C_0201_0603Metric"
 			(at 168.6052 68.58 0)
 			(effects
@@
 			)
 		)
-		(property "Footprint" ""
+		(property "Footprint" "Resistor_SMD:R_0201_0603Metric"
 			(at 205.994 129.794 90)
 			(effects
@@
 			)
 		)
-		(property "Footprint" ""
+		(property "Footprint" "Capacitor_SMD:C_0201_0603Metric"
 			(at 196.5452 104.14 0)
 			(effects
@@
 			)
 		)
-		(property "Footprint" ""
+		(property "Footprint" "Connector_PinHeader_1.00mm:PinHeader_1x03_P1.00mm_Vertical_SMD_Pin1Left"
 			(at 153.67 116.84 0)
 			(effects
@@
 			)
 		)
-		(property "Footprint" ""
+		(property "Footprint" "Capacitor_SMD:C_0201_0603Metric"
 			(at 219.4052 85.09 0)
 			(effects
@@
 			)
 		)
-		(property "Footprint" ""
+		(property "Footprint" "Capacitor_SMD:C_0201_0603Metric"
 			(at 65.7352 156.21 0)
 			(effects
@@
 			)
 		)
-		(property "Footprint" ""
+		(property "Footprint" "LED_SMD:LED_0201_0603Metric"
 			(at 213.36 144.78 0)
 			(effects
@@
 			)
 		)
-		(property "Footprint" ""
+		(property "Footprint" "Resistor_SMD:R_0201_0603Metric"
 			(at 73.914 146.304 90)
 			(effects

Commit message: Place Audio tranformers and cleanup routing.    Re-annotate based on geographical layout.
Parts:
- J3: footprint Connector_PinHeader_1.00mm:PinHeader_1x03_P1.00mm_Vertical_SMD_Pin1Left -> Connector_PinHeader_1.00mm:PinHeader_1x03_P1.00mm_Vertical; now fitted; now in the parts list
Changed lines of the file:
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@@
 		(unit 1)
 		(exclude_from_sim no)
-		(in_bom no)
+		(in_bom yes)
 		(on_board yes)
-		(dnp yes)
+		(dnp no)
 		(fields_autoplaced yes)
 		(property "Reference" "J3"
@@
 			)
 		)
-		(property "Footprint" "Connector_PinHeader_1.00mm:PinHeader_1x03_P1.00mm_Vertical_SMD_Pin1Left"
+		(property "Footprint" "Connector_PinHeader_1.00mm:PinHeader_1x03_P1.00mm_Vertical"
 			(at 153.67 116.84 0)
 			(effects

Commit message: Move Radio interface onto it's own sheet, Add mounting holes and case outline
Parts:
- renumbered C11 to C1, C19 to C10, C14 to C11, C18 to C4, C13 to C7, C15 to C8, C12 to C9, D3 to D2, D4 to D3, J3 to J1, R16 to R10, R18 to R3, R15 to R5, R17 to R7, U8 to U2, U9 to U3
Changed lines of the file:
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@@
 		(on_board yes)
 		(dnp no)
-		(property "Reference" "C19"
+		(property "Reference" "C10"
 			(at 224.028 78.994 0)
 			(effects
@@
 			(project "digital-mode-radio-interface"
 				(path "/a0d4bcf6-6cac-4e92-853e-9083f008b231/6f837d65-f274-4a4b-8cdc-594a0aab134b"
-					(reference "C19")
+					(reference "C10")
 					(unit 1)
 				)
@@
 		(dnp no)
 		(fields_autoplaced yes)
-		(property "Reference" "D3"
+		(property "Reference" "D2"
 			(at 214.9475 123.19 0)
 			(effects
@@
 			(project "digital-mode-radio-interface"
 				(path "/a0d4bcf6-6cac-4e92-853e-9083f008b231/6f837d65-f274-4a4b-8cdc-594a0aab134b"
-					(reference "D3")
+					(reference "D2")
 					(unit 1)
 				)
@@
 		(on_board yes)
 		(dnp no)
-		(property "Reference" "R17"
+		(property "Reference" "R7"
 			(at 73.66 161.544 90)
 			(effects
@@
 			(project "digital-mode-radio-interface"
 				(path "/a0d4bcf6-6cac-4e92-853e-9083f008b231/6f837d65-f274-4a4b-8cdc-594a0aab134b"
-					(reference "R17")
+					(reference "R7")
 					(unit 1)
 				)
@@
 		(on_board yes)
 		(dnp no)
-		(property "Reference" "C15"
+		(property "Reference" "C8"
 			(at 186.436 62.738 0)
 			(effects
@@
 			(project "digital-mode-radio-interface"
 				(path "/a0d4bcf6-6cac-4e92-853e-9083f008b231/6f837d65-f274-4a4b-8cdc-594a0aab134b"
-					(reference "C15")
+					(reference "C8")
 					(unit 1)
 				)
@@
 		(on_board yes)
 		(dnp no)
-		(property "Reference" "R16"
+		(property "Reference" "R10"
 			(at 205.232 142.494 90)
 			(effects
@@
 			(project "digital-mode-radio-interface"
 				(path "/a0d4bcf6-6cac-4e92-853e-9083f008b231/6f837d65-f274-4a4b-8cdc-594a0aab134b"
-					(reference "R16")
+					(reference "R10")
 					(unit 1)
 				)
@@
 		(dnp no)
 		(fields_autoplaced yes)
-		(property "Reference" "U8"
+		(property "Reference" "U2"
 			(at 127 43.18 0)
 			(effects
@@
 			(project "digital-mode-radio-interface"
 				(path "/a0d4bcf6-6cac-4e92-853e-9083f008b231/6f837d65-f274-4a4b-8cdc-594a0aab134b"
-					(reference "U8")
+					(reference "U2")
 					(unit 1)
 				)
@@
 		(on_board yes)
 		(dnp no)
-		(property "Reference" "C14"
+		(property "Reference" "C11"
 			(at 174.752 62.484 0)
 			(effects
@@
 			(project "digital-mode-radio-interface"
 				(path "/a0d4bcf6-6cac-4e92-853e-9083f008b231/6f837d65-f274-4a4b-8cdc-594a0aab134b"
-					(reference "C14")
+					(reference "C11")
 					(unit 1)
 				)
@@
 		(on_board yes)
 		(dnp yes)
-		(property "Reference" "U9"
+		(property "Reference" "U3"
 			(at 186.69 109.6362 0)
 			(effects
@@
 			(project "digital-mode-radio-interface"
 				(path "/a0d4bcf6-6cac-4e92-853e-9083f008b231/6f837d65-f274-4a4b-8cdc-594a0aab134b"
-					(reference "U9")
+					(reference "U3")
 					(unit 1)
 				)
@@
 		(on_board yes)
 		(dnp no)
-		(property "Reference" "C13"
+		(property "Reference" "C7"
 			(at 161.036 62.738 0)
 			(effects
@@
 			(project "digital-mode-radio-interface"
 				(path "/a0d4bcf6-6cac-4e92-853e-9083f008b231/6f837d65-f274-4a4b-8cdc-594a0aab134b"
-					(reference "C13")
+					(reference "C7")
 					(unit 1)
 				)
@@
 		(on_board yes)
 		(dnp no)
-		(property "Reference" "R15"
+		(property "Reference" "R5"
 			(at 205.232 128.778 90)
 			(effects
@@
 			(project "digital-mode-radio-interface"
 				(path "/a0d4bcf6-6cac-4e92-853e-9083f008b231/6f837d65-f274-4a4b-8cdc-594a0aab134b"
-					(reference "R15")
+					(reference "R5")
 					(unit 1)
 				)
@@
 		(on_board yes)
 		(dnp no)
-		(property "Reference" "C11"
+		(property "Reference" "C1"
 			(at 189.738 98.044 0)
 			(effects
@@
 			(project "digital-mode-radio-interface"
 				(path "/a0d4bcf6-6cac-4e92-853e-9083f008b231/6f837d65-f274-4a4b-8cdc-594a0aab134b"
-					(reference "C11")
+					(reference "C1")
 					(unit 1)
 				)
@@
 		(dnp no)
 		(fields_autoplaced yes)
-		(property "Reference" "J3"
+		(property "Reference" "J1"
 			(at 154.94 115.5699 0)
 			(effects
@@
 			(project "digital-mode-radio-interface"
 				(path "/a0d4bcf6-6cac-4e92-853e-9083f008b231/6f837d65-f274-4a4b-8cdc-594a0aab134b"
-					(reference "J3")
+					(reference "J1")
 					(unit 1)
 				)
@@
 		(on_board yes)
 		(dnp no)
-		(property "Reference" "C12"
+		(property "Reference" "C9"
 			(at 212.598 78.994 0)
 			(effects
@@
 			(project "digital-mode-radio-interface"
 				(path "/a0d4bcf6-6cac-4e92-853e-9083f008b231/6f837d65-f274-4a4b-8cdc-594a0aab134b"
-					(reference "C12")
+					(reference "C9")
 					(unit 1)
 				)
@@
 		(on_board yes)
 		(dnp no)
-		(property "Reference" "C18"
+		(property "Reference" "C4"
 			(at 58.928 150.114 0)
 			(effects
@@
 			(project "digital-mode-radio-interface"
 				(path "/a0d4bcf6-6cac-4e92-853e-9083f008b231/6f837d65-f274-4a4b-8cdc-594a0aab134b"
-					(reference "C18")
+					(reference "C4")
 					(unit 1)
 				)
@@
 		(dnp no)
 		(fields_autoplaced yes)
-		(property "Reference" "D4"
+		(property "Reference" "D3"
 			(at 214.9475 137.16 0)
 			(effects
@@
 			(project "digital-mode-radio-interface"
 				(path "/a0d4bcf6-6cac-4e92-853e-9083f008b231/6f837d65-f274-4a4b-8cdc-594a0aab134b"
-					(reference "D4")
+					(reference "D3")
 					(unit 1)
 				)
@@
 		(on_board yes)
 		(dnp no)
-		(property "Reference" "R18"
+		(property "Reference" "R3"
 			(at 73.406 144.78 90)
 			(effects
@@
 			(project "digital-mode-radio-interface"
 				(path "/a0d4bcf6-6cac-4e92-853e-9083f008b231/6f837d65-f274-4a4b-8cdc-594a0aab134b"
-					(reference "R18")
-					(unit 1)
-				)
+					(reference "R3")
+					(unit 1)
+				)
