File: radio_iface.kicad_sch (KiCad schematic)
At the start: 3 parts, among them J3 Conn_01x09_Socket

Commit message: kiCAD 9.0
Changed lines of the file:
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@@
 (kicad_sch
-	(version 20231120)
+	(version 20250114)
 	(generator "eeschema")
-	(generator_version "8.0")
+	(generator_version "9.0")
 	(paper "USLetter")
 	(title_block
